File: Hardware/Main_Board.sch (EAGLE design)
At the start: 22 parts, among them Q1 4MHz, Q2 32.768KHz, Q3 BD135, U1 DS1307Z+, U2 PIC16F876-20/SP, U3 LM35DZ

Commit message: Added display command signal names, a stabilization capacitor and a missing pull-up on the RTC SQW/OUT signal.
Parts:
- added C3: 100n, capacitor-wima:C5/3.5
- added R9: 10K, resistor:R-EU_0207/12
Connections:
- net +5V: now also C3.2, R9.1
- net GND: now also C3.1
- net N$10: now also R9.2
Other:
- note added: "DB4"
- note added: "DB5"
- note added: "DB6"
- note added: "DB7"
- note added: "E"
- note added: "LED-"
- note added: "R/S"
- note added: "R/W"
Changed lines of the file:
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@@
 <setting verticaltext="up"/>
 </settings>
-<grid distance="0.1" unitdist="inch" unit="inch" style="lines" multiple="1" display="yes" altdistance="0.01" altunitdist="inch" altunit="inch"/>
+<grid distance="0.1" unitdist="inch" unit="inch" style="lines" multiple="1" display="no" altdistance="0.01" altunitdist="inch" altunit="inch"/>
 <layers>
 <layer number="1" name="Top" color="4" fill="1" visible="no" active="no"/>
@@
 <part name="P+9" library="supply1" deviceset="+5V" device=""/>
 <part name="GND11" library="supply1" deviceset="GND" device=""/>
+<part name="C3" library="capacitor-wima" deviceset="C" device="5/3.5" value="100n"/>
+<part name="R9" library="resistor" deviceset="R-EU_" device="0207/12" value="10K"/>
+<part name="P+10" library="supply1" deviceset="+5V" device=""/>
 </parts>
 <sheets>
@@
 <text x="170.18" y="73.66" size="1.778" layer="91" rot="R180">V0</text>
 <text x="105.41" y="45.72" size="1.778" layer="91">BUZZER</text>
+<text x="-22.86" y="43.18" size="1.778" layer="91">DB4</text>
+<text x="-22.86" y="40.64" size="1.778" layer="91">DB5</text>
+<text x="-22.86" y="38.1" size="1.778" layer="91">DB6</text>
+<text x="-22.86" y="35.56" size="1.778" layer="91">DB7</text>
+<text x="-22.86" y="45.72" size="1.778" layer="91">E</text>
+<text x="-22.86" y="48.26" size="1.778" layer="91">R/S</text>
+<text x="-22.86" y="50.8" size="1.778" layer="91">R/W</text>
+<text x="-22.86" y="33.02" size="1.778" layer="91">LED-</text>
 </plain>
 <instances>
@@
 <instance part="GND6" gate="1" x="154.94" y="106.68" rot="R270"/>
 <instance part="P+5" gate="1" x="180.34" y="106.68" rot="R270"/>
-<instance part="GND7" gate="1" x="96.52" y="25.4" rot="R90"/>
-<instance part="P+6" gate="1" x="104.14" y="17.78" rot="R270"/>
+<instance part="GND7" gate="1" x="119.38" y="25.4" rot="R90"/>
+<instance part="P+6" gate="1" x="121.92" y="17.78" rot="R270"/>
 <instance part="SG1" gate="G$1" x="99.06" y="43.18"/>
 <instance part="JP1" gate="A" x="91.44" y="10.16" smashed="yes" rot="R270">
@@
 <instance part="P+9" gate="1" x="60.96" y="119.38" rot="MR270"/>
 <instance part="GND11" gate="1" x="60.96" y="114.3" rot="R270"/>
+<instance part="C3" gate="G$1" x="109.22" y="22.86"/>
+<instance part="R9" gate="G$1" x="124.46" y="111.76" rot="R90"/>
+<instance part="P+10" gate="1" x="124.46" y="101.6" rot="R180"/>
 </instances>
 <busses>
@@
 </segment>
 <segment>
-<wire x1="93.98" y1="12.7" x2="93.98" y2="25.4" width="0.1524" layer="91"/>
-<pinref part="GND7" gate="1" pin="GND"/>
-<pinref part="JP1" gate="A" pin="2"/>
-</segment>
-<segment>
 <pinref part="GND8" gate="1" pin="GND"/>
 <pinref part="R5" gate="G$1" pin="1"/>
@@
 <pinref part="GND5" gate="1" pin="GND"/>
 <wire x1="104.14" y1="40.64" x2="106.68" y2="40.64" width="0.1524" layer="91"/>
+</segment>
+<segment>
+<pinref part="GND7" gate="1" pin="GND"/>
+<wire x1="116.84" y1="25.4" x2="109.22" y2="25.4" width="0.1524" layer="91"/>
+<pinref part="JP1" gate="A" pin="2"/>
+<wire x1="109.22" y1="25.4" x2="93.98" y2="25.4" width="0.1524" layer="91"/>
+<wire x1="93.98" y1="25.4" x2="93.98" y2="12.7" width="0.1524" layer="91"/>
+<pinref part="C3" gate="G$1" pin="1"/>
+<junction x="109.22" y="25.4"/>
 </segment>
 </net>
@@
 <segment>
 <pinref part="P+6" gate="1" pin="+5V"/>
-<wire x1="101.6" y1="17.78" x2="96.52" y2="17.78" width="0.1524" layer="91"/>
+<wire x1="119.38" y1="17.78" x2="109.22" y2="17.78" width="0.1524" layer="91"/>
+<wire x1="109.22" y1="17.78" x2="96.52" y2="17.78" width="0.1524" layer="91"/>
 <wire x1="96.52" y1="17.78" x2="96.52" y2="12.7" width="0.1524" layer="91"/>
 <pinref part="JP1" gate="A" pin="1"/>
+<pinref part="C3" gate="G$1" pin="2"/>
+<junction x="109.22" y="17.78"/>
 </segment>
 <segment>
@@
 <pinref part="U3" gate="A" pin="+VS"/>
 <wire x1="63.5" y1="119.38" x2="68.58" y2="119.38" width="0.1524" layer="91"/>
+</segment>
+<segment>
+<pinref part="P+10" gate="1" pin="+5V"/>
+<pinref part="R9" gate="G$1" pin="1"/>
+<wire x1="124.46" y1="104.14" x2="124.46" y2="106.68" width="0.1524" layer="91"/>
 </segment>
 </net>
@@
 <wire x1="86.36" y1="58.42" x2="111.76" y2="58.42" width="0.1524" layer="91"/>
 <wire x1="111.76" y1="58.42" x2="111.76" y2="119.38" width="0.1524" layer="91"/>
-<wire x1="111.76" y1="119.38" x2="205.74" y2="119.38" width="0.1524" layer="91"/>
+<wire x1="111.76" y1="119.38" x2="124.46" y2="119.38" width="0.1524" layer="91"/>
+<wire x1="124.46" y1="119.38" x2="205.74" y2="119.38" width="0.1524" layer="91"/>
 <wire x1="205.74" y1="119.38" x2="205.74" y2="43.18" width="0.1524" layer="91"/>
+<pinref part="R9" gate="G$1" pin="2"/>
+<wire x1="124.46" y1="116.84" x2="124.46" y2="119.38" width="0.1524" layer="91"/>
+<junction x="124.46" y="119.38"/>
 </segment>
 </net>
@@
 <segment>
 <pinref part="U2" gate="A" pin="RC5/SDO"/>
-<wire x1="86.36" y1="30.48" x2="109.22" y2="30.48" width="0.1524" layer="91"/>
-<wire x1="109.22" y1="30.48" x2="109.22" y2="-2.54" width="0.1524" layer="91"/>
+<wire x1="86.36" y1="30.48" x2="129.54" y2="30.48" width="0.1524" layer="91"/>
+<wire x1="129.54" y1="30.48" x2="129.54" y2="-2.54" width="0.1524" layer="91"/>
 <pinref part="R8" gate="G$1" pin="2"/>
-<wire x1="17.78" y1="-2.54" x2="109.22" y2="-2.54" width="0.1524" layer="91"/>
-</segment>
-</net>
+<wire x1="17.78" y1="-2.54" x2="129.54" y2="-2.54" width="0.1524" layer="91"/>
+</segment>
+</net>

Commit message: Changed some signal to ease routing.
Parts:
- removed JP2: DISPLAY_COMMAND, pinhead:PINHD-1X8
- added JP3: DISPLAY_COMMAND, pinhead:PINHD-1X8
Connections:
- net +5V: now also JP5.3, R4.A; no longer JP5.1, R4.E
- net GND: now also JP5.1, R4.E; no longer JP5.3, R4.A
- net N$11: now also JP3.1; no longer JP2.8
- net N$12: now also JP3.2; no longer JP2.7
- net N$13: now also JP3.3; no longer JP2.6
- net N$14: now also JP3.4; no longer JP2.5
- net N$15: now also JP3.5; no longer JP2.4
- net N$16: now also JP3.6; no longer JP2.3
- net N$17: now also JP3.7; no longer JP2.2
- net N$23: now also JP3.8; no longer JP2.1
Changed lines of the file:
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@@
 <part name="P+4" library="supply1" deviceset="+5V" device=""/>
 <part name="GND5" library="supply1" deviceset="GND" device=""/>
-<part name="JP2" library="pinhead" deviceset="PINHD-1X8" device="" value="DISPLAY_COMMAND"/>
 <part name="R4" library="resistor" deviceset="R-TRIMM" device="3339P" value="10K"/>
 <part name="GND6" library="supply1" deviceset="GND" device=""/>
@@
 <part name="R6" library="resistor" deviceset="R-EU_" device="0207/12" value="10K"/>
 <part name="GND9" library="supply1" deviceset="GND" device=""/>
-<part name="P+8" library="supply1" deviceset="+5V" device=""/>
 <part name="Q3" library="transistor-power" deviceset="BD139" device="" value="BD135"/>
 <part name="R7" library="resistor" deviceset="R-EU_" device="0207/12" value="12/0.5W"/>
@@
 <part name="R9" library="resistor" deviceset="R-EU_" device="0207/12" value="10K"/>
 <part name="P+10" library="supply1" deviceset="+5V" device=""/>
+<part name="JP3" library="pinhead" deviceset="PINHD-1X8" device="" value="DISPLAY_COMMAND"/>
 </parts>
 <sheets>
@@
 <instance part="P+4" gate="1" x="10.16" y="76.2"/>
 <instance part="GND5" gate="1" x="109.22" y="40.64" rot="R90"/>
-<instance part="JP2" gate="A" x="-15.24" y="43.18" rot="R180"/>
 <instance part="R4" gate="G$1" x="167.64" y="106.68" rot="R270"/>
-<instance part="GND6" gate="1" x="154.94" y="106.68" rot="R270"/>
-<instance part="P+5" gate="1" x="180.34" y="106.68" rot="R270"/>
+<instance part="GND6" gate="1" x="180.34" y="106.68" rot="R90"/>
+<instance part="P+5" gate="1" x="154.94" y="106.68" rot="R90"/>
 <instance part="GND7" gate="1" x="119.38" y="25.4" rot="R90"/>
 <instance part="P+6" gate="1" x="121.92" y="17.78" rot="R270"/>
@@
 <instance part="R6" gate="G$1" x="142.24" y="93.98" rot="R270"/>
 <instance part="GND9" gate="1" x="142.24" y="104.14" rot="R180"/>
-<instance part="P+8" gate="1" x="162.56" y="93.98"/>
 <instance part="Q3" gate="1" x="0" y="-2.54" rot="MR0"/>
 <instance part="R7" gate="G$1" x="-2.54" y="12.7" rot="R270"/>
@@
 <instance part="R9" gate="G$1" x="124.46" y="111.76" rot="R90"/>
 <instance part="P+10" gate="1" x="124.46" y="101.6" rot="R180"/>
+<instance part="JP3" gate="A" x="-10.16" y="40.64" smashed="yes">
+<attribute name="NAME" x="-16.51" y="53.975" size="1.778" layer="95"/>
+<attribute name="VALUE" x="-31.75" y="27.94" size="1.778" layer="96"/>
+</instance>
 </instances>
 <busses>
@@
 </segment>
 <segment>
-<pinref part="GND6" gate="1" pin="GND"/>
-<pinref part="R4" gate="G$1" pin="A"/>
-<wire x1="157.48" y1="106.68" x2="160.02" y2="106.68" width="0.1524" layer="91"/>
-<wire x1="160.02" y1="106.68" x2="162.56" y2="106.68" width="0.1524" layer="91"/>
-<wire x1="160.02" y1="106.68" x2="160.02" y2="101.6" width="0.1524" layer="91"/>
-<junction x="160.02" y="106.68"/>
-<wire x1="160.02" y1="101.6" x2="165.1" y2="101.6" width="0.1524" layer="91"/>
-<wire x1="165.1" y1="101.6" x2="165.1" y2="78.74" width="0.1524" layer="91"/>
-<pinref part="JP5" gate="A" pin="3"/>
-</segment>
-<segment>
 <pinref part="GND8" gate="1" pin="GND"/>
 <pinref part="R5" gate="G$1" pin="1"/>
@@
 <pinref part="C3" gate="G$1" pin="1"/>
 <junction x="109.22" y="25.4"/>
+</segment>
+<segment>
+<pinref part="R4" gate="G$1" pin="E"/>
+<wire x1="175.26" y1="106.68" x2="172.72" y2="106.68" width="0.1524" layer="91"/>
+<wire x1="175.26" y1="106.68" x2="175.26" y2="101.6" width="0.1524" layer="91"/>
+<wire x1="175.26" y1="101.6" x2="170.18" y2="101.6" width="0.1524" layer="91"/>
+<wire x1="170.18" y1="101.6" x2="170.18" y2="78.74" width="0.1524" layer="91"/>
+<pinref part="JP5" gate="A" pin="1"/>
+<pinref part="GND6" gate="1" pin="GND"/>
+<wire x1="175.26" y1="106.68" x2="177.8" y2="106.68" width="0.1524" layer="91"/>
+<junction x="175.26" y="106.68"/>
 </segment>
 </net>
@@
 </segment>
 <segment>
-<pinref part="P+5" gate="1" pin="+5V"/>
-<pinref part="R4" gate="G$1" pin="E"/>
-<wire x1="177.8" y1="106.68" x2="175.26" y2="106.68" width="0.1524" layer="91"/>
-<wire x1="175.26" y1="106.68" x2="172.72" y2="106.68" width="0.1524" layer="91"/>
-<wire x1="175.26" y1="106.68" x2="175.26" y2="101.6" width="0.1524" layer="91"/>
-<junction x="175.26" y="106.68"/>
-<wire x1="175.26" y1="101.6" x2="170.18" y2="101.6" width="0.1524" layer="91"/>
-<wire x1="170.18" y1="101.6" x2="170.18" y2="78.74" width="0.1524" layer="91"/>
-<pinref part="JP5" gate="A" pin="1"/>
-</segment>
-<segment>
 <pinref part="P+6" gate="1" pin="+5V"/>
 <wire x1="119.38" y1="17.78" x2="109.22" y2="17.78" width="0.1524" layer="91"/>
@@
 </segment>
 <segment>
-<pinref part="JP5" gate="A" pin="4"/>
-<pinref part="P+8" gate="1" pin="+5V"/>
-<wire x1="162.56" y1="78.74" x2="162.56" y2="91.44" width="0.1524" layer="91"/>
-</segment>
-<segment>
 <pinref part="P+9" gate="1" pin="+5V"/>
 <pinref part="U3" gate="A" pin="+VS"/>
@@
 <pinref part="R9" gate="G$1" pin="1"/>
 <wire x1="124.46" y1="104.14" x2="124.46" y2="106.68" width="0.1524" layer="91"/>
+</segment>
+<segment>
+<pinref part="R4" gate="G$1" pin="A"/>
+<wire x1="160.02" y1="106.68" x2="162.56" y2="106.68" width="0.1524" layer="91"/>
+<wire x1="160.02" y1="106.68" x2="160.02" y2="101.6" width="0.1524" layer="91"/>
+<wire x1="160.02" y1="101.6" x2="165.1" y2="101.6" width="0.1524" layer="91"/>
+<wire x1="165.1" y1="101.6" x2="165.1" y2="86.36" width="0.1524" layer="91"/>
+<pinref part="JP5" gate="A" pin="3"/>
+<pinref part="P+5" gate="1" pin="+5V"/>
+<wire x1="165.1" y1="86.36" x2="165.1" y2="78.74" width="0.1524" layer="91"/>
+<wire x1="160.02" y1="106.68" x2="157.48" y2="106.68" width="0.1524" layer="91"/>
+<junction x="160.02" y="106.68"/>
+<pinref part="JP5" gate="A" pin="4"/>
+<wire x1="162.56" y1="78.74" x2="162.56" y2="86.36" width="0.1524" layer="91"/>
+<wire x1="162.56" y1="86.36" x2="165.1" y2="86.36" width="0.1524" layer="91"/>
+<junction x="165.1" y="86.36"/>
 </segment>
 </net>
@@
 <segment>
 <pinref part="U2" gate="A" pin="RB1"/>
-<pinref part="JP2" gate="A" pin="8"/>
 <wire x1="20.32" y1="50.8" x2="-12.7" y2="50.8" width="0.1524" layer="91"/>
+<pinref part="JP3" gate="A" pin="1"/>
 </segment>
 </net>
@@
 <segment>
 <pinref part="U2" gate="A" pin="RB2"/>
-<pinref part="JP2" gate="A" pin="7"/>
 <wire x1="20.32" y1="48.26" x2="-12.7" y2="48.26" width="0.1524" layer="91"/>
+<pinref part="JP3" gate="A" pin="2"/>
 </segment>
 </net>
@@
 <segment>
 <pinref part="U2" gate="A" pin="RB3/PGM"/>
-<pinref part="JP2" gate="A" pin="6"/>
 <wire x1="20.32" y1="45.72" x2="-12.7" y2="45.72" width="0.1524" layer="91"/>
+<pinref part="JP3" gate="A" pin="3"/>
 </segment>
 </net>
@@
 <segment>
 <pinref part="U2" gate="A" pin="RB4"/>
-<pinref part="JP2" gate="A" pin="5"/>
 <wire x1="20.32" y1="43.18" x2="-12.7" y2="43.18" width="0.1524" layer="91"/>
+<pinref part="JP3" gate="A" pin="4"/>
 </segment>
 </net>
@@
 <segment>
 <pinref part="U2" gate="A" pin="RB5"/>
-<pinref part="JP2" gate="A" pin="4"/>
 <wire x1="20.32" y1="40.64" x2="-12.7" y2="40.64" width="0.1524" layer="91"/>
+<pinref part="JP3" gate="A" pin="5"/>
 </segment>
 </net>
@@
 <segment>
 <pinref part="U2" gate="A" pin="RB6/PGC"/>
-<pinref part="JP2" gate="A" pin="3"/>
 <wire x1="20.32" y1="38.1" x2="-12.7" y2="38.1" width="0.1524" layer="91"/>
+<pinref part="JP3" gate="A" pin="6"/>
 </segment>
 </net>
@@
 <segment>
 <pinref part="U2" gate="A" pin="RB7/PGD"/>
-<pinref part="JP2" gate="A" pin="2"/>
 <wire x1="20.32" y1="35.56" x2="-12.7" y2="35.56" width="0.1524" layer="91"/>
+<pinref part="JP3" gate="A" pin="7"/>
 </segment>
 </net>
@@
 <net name="N$23" class="0">
 <segment>
-<pinref part="JP2" gate="A" pin="1"/>
 <wire x1="-12.7" y1="33.02" x2="-2.54" y2="33.02" width="0.1524" layer="91"/>
 <pinref part="R7" gate="G$1" pin="1"/>
 <wire x1="-2.54" y1="33.02" x2="-2.54" y2="17.78" width="0.1524" layer="91"/>
-</segment>
-</net>
+<pinref part="JP3" gate="A" pin="8"/>
+</segment>
+</net>

Commit message: Changed the display backlight driver transistor base resistor (R8) to 1Kohm because 100Ohm were generating Read-Modify-Write errors on the PIC port.
Parts:
- R8: value 100 -> 1K
Changed lines of the file:
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@@
 <part name="Q3" library="transistor-power" deviceset="BD139" device="" value="BD135"/>
 <part name="R7" library="resistor" deviceset="R-EU_" device="0207/12" value="12/0.5W"/>
-<part name="R8" library="resistor" deviceset="R-EU_" device="0207/12" value="100"/>
+<part name="R8" library="resistor" deviceset="R-EU_" device="0207/12" value="1K"/>
 <part name="GND10" library="supply1" deviceset="GND" device=""/>
 <part name="U3" library="LM35DZ" deviceset="LM35DZ" device=""/>

Commit message: Added a decoupling resistor on the temperature sensor output as the microcontroller ADC input has a too high capacitance.
Parts:
- added R10: 2.2K, resistor:R-EU_0207/12
Connections:
- new net N$28: R10.1, U3.VOUT
- net N$27: now also R10.2; no longer U3.VOUT
Changed lines of the file:
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@@
 <part name="P+10" library="supply1" deviceset="+5V" device=""/>
 <part name="JP3" library="pinhead" deviceset="PINHD-1X8" device="" value="DISPLAY_COMMAND"/>
+<part name="R10" library="resistor" deviceset="R-EU_" device="0207/12" value="2.2K"/>
 </parts>
 <sheets>
@@
 <attribute name="VALUE" x="-31.75" y="27.94" size="1.778" layer="96"/>
 </instance>
+<instance part="R10" gate="G$1" x="106.68" y="91.44" rot="R270"/>
 </instances>
 <busses>
@@
 <segment>
 <wire x1="86.36" y1="60.96" x2="106.68" y2="60.96" width="0.1524" layer="91"/>
-<wire x1="106.68" y1="60.96" x2="106.68" y2="119.38" width="0.1524" layer="91"/>
+<wire x1="106.68" y1="60.96" x2="106.68" y2="86.36" width="0.1524" layer="91"/>
+<pinref part="U2" gate="A" pin="RA0/AN0"/>
+<pinref part="R10" gate="G$1" pin="2"/>
+</segment>
+</net>
+<net name="N$28" class="0">
+<segment>
 <pinref part="U3" gate="A" pin="VOUT"/>
 <wire x1="106.68" y1="119.38" x2="104.14" y2="119.38" width="0.1524" layer="91"/>
-<pinref part="U2" gate="A" pin="RA0/AN0"/>
-</segment>
-</net>
+<wire x1="106.68" y1="96.52" x2="106.68" y2="119.38" width="0.1524" layer="91"/>
+<pinref part="R10" gate="G$1" pin="1"/>
+</segment>
+</net>

Commit message: Improved hardware stability by adding decoupling capacitors.
Parts:
- added C4: 100n 25V, rcl:C-EU025-025X050
- added C5: 470n 25V, rcl:C-EU025-025X050
- added C6: 220u 25V, rcl:CPOL-EUE2.5-6
- C1, C2: value 15pF -> 15p 25V
- C3: value 100n -> 100n 25V
Connections:
- net +5V: now also C4.1, C5.1, C6.+
- net GND: now also C4.2, C5.2, C6.-
Other:
- moved on the sheet: C3, R4, R9, U3
